Commit message: Update dimensions and position in my_robot.urdf
made dimentions more accurate

File: scripts/my_robot.urdf (robot description, URDF)
Before this commit: robot mren_robot, 2 links, 1 joints
Links:
- link base_link: geometry visual box size=0.33 0.33 0.1
- link laser: geometry visual cylinder length=0.06 radius=0.0325
Joints:
- joint laser_joint: origin xyz=0.1 0 0.05 rpy=0 0 0 -> xyz=0.05 0.05 0.1 rpy=0 0 0

Commit message: thursday update

File: scripts/my_robot.urdf (robot description, URDF)
Before this commit: robot mren_robot, 2 links, 1 joints
Links:
- removed link laser
- added link laser_frame; visual cylinder length=0.06 radius=0.0325
Joints:
- joint laser_joint: child laser -> laser_frame

Commit message: not done

File: scripts/my_robot.urdf (robot description, URDF)
Before this commit: robot mren_robot, 2 links, 1 joints
Links:
- removed link laser_frame
- added link laser; visual cylinder length=0.06 radius=0.0325
Joints:
- joint laser_joint: child laser_frame -> laser
